Commit message: Add depth camera from components_snippets and add enable_depth_camera_visual

File: rotors_description/urdf/component_snippets.xacro (robot description, xacro)
@@ -597,5 +597,5 @@
   <!-- Macro to add a depth camera on the VI-sensor. -->
   <xacro:macro name="vi_sensor_depth_macro"
-    params="namespace parent_link camera_suffix frame_rate max_range *origin">
+    params="namespace parent_link camera_suffix frame_rate max_range enable_depth_camera_visual *geometry *origin">
     <link name="${namespace}/camera_${camera_suffix}_link">
       <collision>
@@ -605,4 +605,13 @@
         </geometry>
       </collision>
+      <xacro:if value="${enable_depth_camera_visual}">
+        <visual>
+          <origin xyz="0 0 0" rpy="0 ${pi/2} 0" />
+          <geometry>
+            <xacro:insert_block name="geometry" />
+          </geometry>
+          <material name="red" />
+        </visual>
+      </xacro:if>
       <inertial>
         <mass value="1e-5" />
@@ -665,5 +674,5 @@
   </xacro:macro>
   <!-- VI-Sensor Macro -->
-  <xacro:macro name="vi_sensor_macro" params="namespace parent_link enable_cameras enable_depth enable_ground_truth *origin">
+  <xacro:macro name="vi_sensor_macro" params="namespace parent_link enable_cameras enable_depth enable_depth_camera_visual enable_ground_truth *origin">
     <!-- Vi Sensor Link -->
     <link name="${namespace}/vi_sensor_link">
@@ -697,5 +706,5 @@
         namespace="${namespace}" parent_link="${namespace}/vi_sensor_link"
         frame_rate="30.0" origin_offset_x="0.015" baseline_y="${0.055*2}"
-        origin_offset_z="0.0065" max_range="30.0">
+        origin_offset_z="0.0065" max_range="30.0" enable_depth_camera_visual="${enable_depth_camera_visual}">
       </xacro:vi_sensor_stereo_camera_macro>
     </xacro:if>

File: rotors_description/urdf/firefly.xacro (robot description, xacro)
@@ -184,5 +184,8 @@
     <xacro:insert_block name="rotor_inertia" />
   </xacro:vertical_rotor>
-  <xacro:camera_macro
+  <!--  -->
+  <!-- CUSTOM EDITS BELOW -->
+  <!--  -->
+  <!-- <xacro:camera_macro
     namespace="${namespace}"
     parent_link="${namespace}/base_link"
@@ -199,5 +202,11 @@
     enable_visual="true">
     <box size="0.05 0.05 0.02" />
-    <origin xyz="0 0 ${-arm_length/4}" rpy="0 ${pi/4} 0" />
-  </xacro:camera_macro>
+    <origin xyz="0 0 ${-arm_length/4}" rpy="0 ${pi/2} 0" />
+  </xacro:camera_macro> -->
+  <xacro:vi_sensor_depth_macro
+        namespace="${namespace}" parent_link="${namespace}/base_link"
+        camera_suffix="depth" frame_rate="30.0" max_range="10.0" enable_depth_camera_visual="true">
+        <box size="0.05 0.05 0.02" />
+        <origin xyz="0 0 ${-arm_length/4}" rpy="0 ${pi/2} 0" />
+  </xacro:vi_sensor_depth_macro>
 </robot>
