Commit message: Update Custom Branch

File: rotors_description/urdf/firefly.xacro (robot description, xacro)
@@ -184,3 +184,20 @@
     <xacro:insert_block name="rotor_inertia" />
   </xacro:vertical_rotor>
+  <xacro:camera_macro
+    namespace="${namespace}"
+    parent_link="${namespace}/base_link"
+    camera_suffix="nadir"
+    frame_rate="60.0"
+    horizontal_fov="2"
+    image_width="752"
+    image_height="480"
+    image_format="L8"
+    min_distance="0.02"
+    max_distance="50"
+    noise_mean="0.0"
+    noise_stddev="0.007"
+    enable_visual="true">
+    <box size="0.05 0.05 0.02" />
+    <origin xyz="0 0 ${-arm_length/4}" rpy="0 ${pi/4} 0" />
+  </xacro:camera_macro>
 </robot>

Commit message: Update firefly mesh and readme

File: rotors_description/urdf/firefly.xacro (robot description, xacro)
@@ -16,5 +16,6 @@
   limitations under the License.
 -->
-<robot name="firefly" xmlns:xacro="http://ros.org/wiki/xacro">
+<robot name="firefly"
+  xmlns:xacro="http://ros.org/wiki/xacro">
   <!-- Properties -->
   <xacro:property name="namespace" value="$(arg namespace)" />
@@ -22,16 +23,28 @@
   <xacro:property name="use_mesh_file" value="true" />
   <xacro:property name="mesh_file" value="package://rotors_description/meshes/firefly.dae" />
-  <xacro:property name="mass" value="1.5" /> <!-- [kg] -->
-  <xacro:property name="body_width" value="0.1" /> <!-- [m] -->
-  <xacro:property name="body_height" value="0.16" /> <!-- [m] -->
-  <xacro:property name="mass_rotor" value="0.005" /> <!-- [kg] -->
-  <xacro:property name="arm_length" value="0.215" /> <!-- [m] -->
-  <xacro:property name="rotor_offset_top" value="0.037" /> <!-- [m] -->
-  <xacro:property name="radius_rotor" value="0.1" /> <!-- [m] -->
-  <xacro:property name="motor_constant" value="8.54858e-06" /> <!-- [kg m/s^2] -->
-  <xacro:property name="moment_constant" value="0.016" /> <!-- [m] -->
-  <xacro:property name="time_constant_up" value="0.0125" /> <!-- [s] -->
-  <xacro:property name="time_constant_down" value="0.025" /> <!-- [s] -->
-  <xacro:property name="max_rot_velocity" value="838" /> <!-- [rad/s] -->
+  <xacro:property name="mass" value="1.5" />
+  <!-- [kg] -->
+  <xacro:property name="body_width" value="0.1" />
+  <!-- [m] -->
+  <xacro:property name="body_height" value="0.06" />
+  <!-- [m] -->
+  <xacro:property name="mass_rotor" value="0.005" />
+  <!-- [kg] -->
+  <xacro:property name="arm_length" value="0.215" />
+  <!-- [m] -->
+  <xacro:property name="rotor_offset_top" value="0.037" />
+  <!-- [m] -->
+  <xacro:property name="radius_rotor" value="0.1" />
+  <!-- [m] -->
+  <xacro:property name="motor_constant" value="8.54858e-06" />
+  <!-- [kg m/s^2] -->
+  <xacro:property name="moment_constant" value="0.016" />
+  <!-- [m] -->
+  <xacro:property name="time_constant_up" value="0.0125" />
+  <!-- [s] -->
+  <xacro:property name="time_constant_down" value="0.025" />
+  <!-- [s] -->
+  <xacro:property name="max_rot_velocity" value="838" />
+  <!-- [rad/s] -->
   <xacro:property name="sin30" value="0.5" />
   <xacro:property name="cos30" value="0.866025403784" />
@@ -40,5 +53,6 @@
   <!-- Property Blocks -->
   <xacro:property name="body_inertia">
-    <inertia ixx="0.0347563" ixy="0.0" ixz="0.0" iyy="0.0458929" iyz="0.0" izz="0.0977" /> <!-- [kg m^2] [kg m^2] [kg m^2] [kg m^2] [kg m^2] [kg m^2] -->
+    <inertia ixx="0.0347563" ixy="0.0" ixz="0.0" iyy="0.0458929" iyz="0.0" izz="0.0977" />
+    <!-- [kg m^2] [kg m^2] [kg m^2] [kg m^2] [kg m^2] [kg m^2] -->
   </xacro:property>
   <!-- inertia of a single rotor, assuming it is a cuboid. Height=3mm, width=15mm -->
@@ -49,136 +63,29 @@
   <xacro:include filename="$(find rotors_description)/urdf/multirotor_base.xacro" />
   <!-- Instantiate multirotor_base_macro once -->
-  <xacro:multirotor_base_macro
-    robot_namespace="${namespace}"
-    mass="${mass}"
-    body_width="${body_width}"
-    body_height="${body_height}"
-    use_mesh_file="${use_mesh_file}"
-    mesh_file="${mesh_file}"
-    >
+  <xacro:multirotor_base_macro robot_namespace="${namespace}" mass="${mass}" body_width="${body_width}" body_height="${body_height}" use_mesh_file="${use_mesh_file}" mesh_file="${mesh_file}">
     <xacro:insert_block name="body_inertia" />
   </xacro:multirotor_base_macro>
   <!-- Instantiate rotors -->
-  <xacro:vertical_rotor
-    robot_namespace="${namespace}"
-    suffix="front_left"
-    direction="ccw"
-    motor_constant="${motor_constant}"
-    moment_constant="${moment_constant}"
-    parent="${namespace}/base_link"
-    mass_rotor="${mass_rotor}"
-    radius_rotor="${radius_rotor}"
-    time_constant_up="${time_constant_up}"
-    time_constant_down="${time_constant_down}"
-    max_rot_velocity="${max_rot_velocity}"
-    motor_number="0"
-    rotor_drag_coefficient="${rotor_drag_coefficient}"
-    rolling_moment_coefficient="${rolling_moment_coefficient}"
-    color="Red"
-    use_own_mesh="false"
-    mesh="">
+  <xacro:vertical_rotor robot_namespace="${namespace}" suffix="front_left" direction="ccw" motor_constant="${motor_constant}" moment_constant="${moment_constant}" parent="${namespace}/base_link" mass_rotor="${mass_rotor}" radius_rotor="${radius_rotor}" time_constant_up="${time_constant_up}" time_constant_down="${time_constant_down}" max_rot_velocity="${max_rot_velocity}" motor_number="0" rotor_drag_coefficient="${rotor_drag_coefficient}" rolling_moment_coefficient="${rolling_moment_coefficient}" color="Red" use_own_mesh="false" mesh="">
     <origin xyz="${cos30*arm_length} ${sin30*arm_length} ${rotor_offset_top}" rpy="0 0 0" />
     <xacro:insert_block name="rotor_inertia" />
   </xacro:vertical_rotor>
-  <xacro:vertical_rotor
-    robot_namespace="${namespace}"
-    suffix="left"
-    direction="cw"
-    motor_constant="${motor_constant}"
-    moment_constant="${moment_constant}"
-    parent="${namespace}/base_link"
-    mass_rotor="${mass_rotor}"
-    radius_rotor="${radius_rotor}"
-    time_constant_up="${time_constant_up}"
-    time_constant_down="${time_constant_down}"
-    max_rot_velocity="${max_rot_velocity}"
-    motor_number="1"
-    rotor_drag_coefficient="${rotor_drag_coefficient}"
-    rolling_moment_coefficient="${rolling_moment_coefficient}"
-    color="Blue"
-    use_own_mesh="false"
-    mesh="">
+  <xacro:vertical_rotor robot_namespace="${namespace}" suffix="left" direction="cw" motor_constant="${motor_constant}" moment_constant="${moment_constant}" parent="${namespace}/base_link" mass_rotor="${mass_rotor}" radius_rotor="${radius_rotor}" time_constant_up="${time_constant_up}" time_constant_down="${time_constant_down}" max_rot_velocity="${max_rot_velocity}" motor_number="1" rotor_drag_coefficient="${rotor_drag_coefficient}" rolling_moment_coefficient="${rolling_moment_coefficient}" color="Blue" use_own_mesh="false" mesh="">
     <origin xyz="0 ${arm_length} ${rotor_offset_top}" rpy="0 0 0" />
     <xacro:insert_block name="rotor_inertia" />
   </xacro:vertical_rotor>
-  <xacro:vertical_rotor robot_namespace="${namespace}"
-    suffix="back_left"
-    direction="ccw"
-    motor_constant="${motor_constant}"
-    moment_constant="${moment_constant}"
-    parent="${namespace}/base_link"
-    mass_rotor="${mass_rotor}"
-    radius_rotor="${radius_rotor}"
-    time_constant_up="${time_constant_up}"
-    time_constant_down="${time_constant_down}"
-    max_rot_velocity="${max_rot_velocity}"
-    motor_number="2"
-    rotor_drag_coefficient="${rotor_drag_coefficient}"
-    rolling_moment_coefficient="${rolling_moment_coefficient}"
-    color="Blue"
-    use_own_mesh="false"
-    mesh="">
+  <xacro:vertical_rotor robot_namespace="${namespace}" suffix="back_left" direction="ccw" motor_constant="${motor_constant}" moment_constant="${moment_constant}" parent="${namespace}/base_link" mass_rotor="${mass_rotor}" radius_rotor="${radius_rotor}" time_constant_up="${time_constant_up}" time_constant_down="${time_constant_down}" max_rot_velocity="${max_rot_velocity}" motor_number="2" rotor_drag_coefficient="${rotor_drag_coefficient}" rolling_moment_coefficient="${rolling_moment_coefficient}" color="Blue" use_own_mesh="false" mesh="">
     <origin xyz="-${cos30*arm_length} ${sin30*arm_length} ${rotor_offset_top}" rpy="0 0 0" />
     <xacro:insert_block name="rotor_inertia" />
   </xacro:vertical_rotor>
-  <xacro:vertical_rotor robot_namespace="${namespace}"
-    suffix="back_right"
-    direction="cw"
-    motor_constant="${motor_constant}"
-    moment_constant="${moment_constant}"
-    parent="${namespace}/base_link"
-    mass_rotor="${mass_rotor}"
-    radius_rotor="${radius_rotor}"
-    time_constant_up="${time_constant_up}"
-    time_constant_down="${time_constant_down}"
-    max_rot_velocity="${max_rot_velocity}"
-    motor_number="3"
-    rotor_drag_coefficient="${rotor_drag_coefficient}"
-    rolling_moment_coefficient="${rolling_moment_coefficient}"
-    color="Blue"
-    use_own_mesh="false"
-    mesh="">
+  <xacro:vertical_rotor robot_namespace="${namespace}" suffix="back_right" direction="cw" motor_constant="${motor_constant}" moment_constant="${moment_constant}" parent="${namespace}/base_link" mass_rotor="${mass_rotor}" radius_rotor="${radius_rotor}" time_constant_up="${time_constant_up}" time_constant_down="${time_constant_down}" max_rot_velocity="${max_rot_velocity}" motor_number="3" rotor_drag_coefficient="${rotor_drag_coefficient}" rolling_moment_coefficient="${rolling_moment_coefficient}" color="Blue" use_own_mesh="false" mesh="">
     <origin xyz="-${cos30*arm_length} -${sin30*arm_length} ${rotor_offset_top}" rpy="0 0 0" />
     <xacro:insert_block name="rotor_inertia" />
   </xacro:vertical_rotor>
-  <xacro:vertical_rotor
-    robot_namespace="${namespace}"
-    suffix="right"
-    direction="ccw"
-    motor_constant="${motor_constant}"
-    moment_constant="${moment_constant}"
-    parent="${namespace}/base_link"
-    mass_rotor="${mass_rotor}"
-    radius_rotor="${radius_rotor}"
-    time_constant_up="${time_constant_up}"
-    time_constant_down="${time_constant_down}"
-    max_rot_velocity="${max_rot_velocity}"
-    motor_number="4"
-    rotor_drag_coefficient="${rotor_drag_coefficient}"
-    rolling_moment_coefficient="${rolling_moment_coefficient}"
-    color="Blue"
-    use_own_mesh="false"
-    mesh="">
+  <xacro:vertical_rotor robot_namespace="${namespace}" suffix="right" direction="ccw" motor_constant="${motor_constant}" moment_constant="${moment_constant}" parent="${namespace}/base_link" mass_rotor="${mass_rotor}" radius_rotor="${radius_rotor}" time_constant_up="${time_constant_up}" time_constant_down="${time_constant_down}" max_rot_velocity="${max_rot_velocity}" motor_number="4" rotor_drag_coefficient="${rotor_drag_coefficient}" rolling_moment_coefficient="${rolling_moment_coefficient}" color="Blue" use_own_mesh="false" mesh="">
     <origin xyz="0 -${arm_length} ${rotor_offset_top}" rpy="0 0 0" />
     <xacro:insert_block name="rotor_inertia" />
   </xacro:vertical_rotor>
-  <xacro:vertical_rotor
-    robot_namespace="${namespace}"
-    suffix="front_right"
-    direction="cw"
-    motor_constant="${motor_constant}"
-    moment_constant="${moment_constant}"
-    parent="${namespace}/base_link"
-    mass_rotor="${mass_rotor}"
-    radius_rotor="${radius_rotor}"
-    time_constant_up="${time_constant_up}"
-    time_constant_down="${time_constant_down}"
-    max_rot_velocity="${max_rot_velocity}"
-    motor_number="5"
-    rotor_drag_coefficient="${rotor_drag_coefficient}"
-    rolling_moment_coefficient="${rolling_moment_coefficient}"
-    color="Red"
-    use_own_mesh="false"
-    mesh="">
+  <xacro:vertical_rotor robot_namespace="${namespace}" suffix="front_right" direction="cw" motor_constant="${motor_constant}" moment_constant="${moment_constant}" parent="${namespace}/base_link" mass_rotor="${mass_rotor}" radius_rotor="${radius_rotor}" time_constant_up="${time_constant_up}" time_constant_down="${time_constant_down}" max_rot_velocity="${max_rot_velocity}" motor_number="5" rotor_drag_coefficient="${rotor_drag_coefficient}" rolling_moment_coefficient="${rolling_moment_coefficient}" color="Red" use_own_mesh="false" mesh="">
     <origin xyz="${cos30*arm_length} -${sin30*arm_length} ${rotor_offset_top}" rpy="0 0 0" />
     <xacro:insert_block name="rotor_inertia" />
@@ -187,26 +94,11 @@
   <!-- CUSTOM EDITS BELOW -->
   <!--  -->
-  <!-- <xacro:camera_macro
-    namespace="${namespace}"
-    parent_link="${namespace}/base_link"
-    camera_suffix="nadir"
-    frame_rate="60.0"
-    horizontal_fov="2"
-    image_width="752"
-    image_height="480"
-    image_format="L8"
-    min_distance="0.02"
-    max_distance="50"
-    noise_mean="0.0"
-    noise_stddev="0.007"
-    enable_visual="true">
+  <!-- <xacro:camera_macro namespace="${namespace}" parent_link="${namespace}/base_link" camera_suffix="nadir" frame_rate="60.0" horizontal_fov="2" image_width="752" image_height="480" image_format="L8" min_distance="0.02" max_distance="50" noise_mean="0.0" noise_stddev="0.007" enable_visual="true">
     <box size="0.05 0.05 0.02" />
     <origin xyz="0 0 ${-arm_length/4}" rpy="0 ${pi/2} 0" />
   </xacro:camera_macro> -->
-  <xacro:vi_sensor_depth_macro
-        namespace="${namespace}" parent_link="${namespace}/base_link"
-        camera_suffix="depth" frame_rate="30.0" max_range="10.0" enable_depth_camera_visual="true">
+  <!-- <xacro:vi_sensor_depth_macro namespace="${namespace}" parent_link="${namespace}/base_link" camera_suffix="depth" frame_rate="30.0" max_range="10.0" enable_depth_camera_visual="true">
         <box size="0.05 0.05 0.02" />
         <origin xyz="0 0 ${-arm_length/4}" rpy="0 ${pi/2} 0" />
-  </xacro:vi_sensor_depth_macro>
+  </xacro:vi_sensor_depth_macro> -->
 </robot>
